Commit message: Finished Task A.3 -Updated tasks.md -Added parameters in diff_params.yaml -Added jsp to launch file (forgot to do in A.2) -Imported yaml parameters into urdf -Updated turtlebot3 urdf to use the yaml parameters

File: nuturtle_description/urdf/turtlebot3_burger.urdf.xacro (robot description, xacro)
@@ -4,4 +4,11 @@
   <xacro:include filename="$(find nuturtle_description)/urdf/common_properties.xacro"/>
   <xacro:include filename="$(find nuturtle_description)/urdf/turtlebot3_burger.gazebo.xacro"/>
+  <!-- Import yaml file -->
+  <xacro:property name="yaml_file" value="$(find nuturtle_description)/config/diff_params.yaml"/>
+  <xacro:property name="yaml" value="${xacro.load_yaml(yaml_file)}"/>
+  <!-- Get properties from yaml file -->
+  <xacro:property name="wheel_radius" value="${yaml['/**']['ros__parameters']['wheel_radius']}"/>
+  <xacro:property name="track_width" value="${yaml['/**']['ros__parameters']['track_width']}"/>
+  <xacro:property name="collision_radius" value="${yaml['/**']['ros__parameters']['collision_radius']}"/>
   <link name="base_footprint"/>
   <joint name="base_joint" type="fixed">
@@ -20,7 +27,14 @@
     <collision>
       <origin xyz="-0.032 0 0.070" rpy="0 0 0"/>
-      <geometry>
-        <box size="0.140 0.140 0.143"/>
-      </geometry>
+      <xacro:if value="${collision_radius &lt; 0}">
+        <geometry>
+          <box size="0.140 0.140 0.143"/>
+        </geometry>
+      </xacro:if>
+      <xacro:if value="${collision_radius &gt;= 0}">
+        <geometry>
+          <cylinder length="0.143" radius="${collision_radius}"/>
+        </geometry>
+      </xacro:if>
     </collision>
     <inertial>
@@ -35,5 +49,5 @@
     <parent link="base_link"/>
     <child link="wheel_left_link"/>
-    <origin xyz="0.0 0.08 0.023" rpy="-1.57 0 0"/>
+    <origin xyz="0.0 ${track_width / 2.0} 0.023" rpy="-1.57 0 0"/>
     <axis xyz="0 0 1"/>
   </joint>
@@ -49,5 +63,5 @@
       <origin xyz="0 0 0" rpy="0 0 0"/>
       <geometry>
-        <cylinder length="0.018" radius="0.033"/>
+        <cylinder length="0.018" radius="${wheel_radius}"/>
       </geometry>
     </collision>
@@ -63,5 +77,5 @@
     <parent link="base_link"/>
     <child link="wheel_right_link"/>
-    <origin xyz="0.0 -0.080 0.023" rpy="-1.57 0 0"/>
+    <origin xyz="0.0 ${-track_width / 2.0} 0.023" rpy="-1.57 0 0"/>
     <axis xyz="0 0 1"/>
   </joint>
@@ -77,5 +91,5 @@
       <origin xyz="0 0 0" rpy="0 0 0"/>
       <geometry>
-        <cylinder length="0.018" radius="0.033"/>
+        <cylinder length="0.018" radius="${wheel_radius}"/>
       </geometry>
     </collision>

Commit message: Finished Task A.4 -Added color argument to xacro -Base link changes based on color argument -Made launch file changes so that each color launches in it's own namespace with its own rviz config

File: nuturtle_description/urdf/turtlebot3_burger.urdf.xacro (robot description, xacro)
@@ -2,6 +2,6 @@
 <!-- This file has been modified from the original version -->
 <robot name="turtlebot3_burger" xmlns:xacro="http://ros.org/wiki/xacro">
-  <xacro:include filename="$(find nuturtle_description)/urdf/common_properties.xacro"/>
-  <xacro:include filename="$(find nuturtle_description)/urdf/turtlebot3_burger.gazebo.xacro"/>
+  <!-- <xacro:include filename="$(find nuturtle_description)/urdf/common_properties.xacro"/>
+  <xacro:include filename="$(find nuturtle_description)/urdf/turtlebot3_burger.gazebo.xacro"/> -->
   <!-- Import yaml file -->
   <xacro:property name="yaml_file" value="$(find nuturtle_description)/config/diff_params.yaml"/>
@@ -11,4 +11,21 @@
   <xacro:property name="track_width" value="${yaml['/**']['ros__parameters']['track_width']}"/>
   <xacro:property name="collision_radius" value="${yaml['/**']['ros__parameters']['collision_radius']}"/>
+  <!-- Color argument -->
+  <xacro:arg name="color" default="purple"/>
+  <xacro:property name="color" value="$(arg color)"/>
+  <!-- Color values -->
+  <material name="purple">
+      <color rgba="0.3 0.16 0.52 1.0"/>
+  </material>
+  <material name="red">
+      <color rgba="1.0 0.0 0.0 1.0"/>
+  </material>
+  <material name="green">
+      <color rgba="0.0 1.0 0.0 1.0"/>
+  </material>
+  <material name="blue">
+      <color rgba="0.0 0.0 1.0 1.0"/>
+  </material>
+  <!-- Robot Description -->
   <link name="base_footprint"/>
   <joint name="base_joint" type="fixed">
@@ -23,5 +40,5 @@
         <mesh filename="package://nuturtle_description/meshes/burger_base.stl" scale="0.001 0.001 0.001"/>
       </geometry>
-      <material name="light_black"/>
+      <material name="${color}"/>
     </visual>
     <collision>
@@ -32,5 +49,5 @@
         </geometry>
       </xacro:if>
-      <xacro:if value="${collision_radius &gt;= 0}">
+      <xacro:if value="${collision_radius &gt; 0}">
         <geometry>
           <cylinder length="0.143" radius="${collision_radius}"/>

Commit message: Finished part A

File: nuturtle_description/urdf/turtlebot3_burger.urdf.xacro (robot description, xacro)
@@ -2,6 +2,5 @@
 <!-- This file has been modified from the original version -->
 <robot name="turtlebot3_burger" xmlns:xacro="http://ros.org/wiki/xacro">
-  <!-- <xacro:include filename="$(find nuturtle_description)/urdf/common_properties.xacro"/>
-  <xacro:include filename="$(find nuturtle_description)/urdf/turtlebot3_burger.gazebo.xacro"/> -->
+  <xacro:include filename="$(find nuturtle_description)/urdf/turtlebot3_burger.gazebo.xacro"/>
   <!-- Import yaml file -->
   <xacro:property name="yaml_file" value="$(find nuturtle_description)/config/diff_params.yaml"/>
@@ -26,4 +25,7 @@
   <material name="blue">
       <color rgba="0.0 0.0 1.0 1.0"/>
+  </material>
+  <material name="dark">
+    <color rgba="0.3 0.3 0.3 1.0"/>
   </material>
   <!-- Robot Description -->
